Commit message: adjust color
Signed-off-by: Daisuke Sato <daisukes@cmu.edu>

File: cabot_description/urdf/sensors/VLP-16_kx.urdf.xacro (robot description, xacro)
@@ -62,4 +62,7 @@
       </collision>
     </link>
+    <gazebo reference="${name}_base_link">
+      <material>Gazebo/Gray</material>
+    </gazebo>
     <joint name="${name}_base_scan_joint" type="fixed">
       <origin xyz="0 0 0.0377" rpy="0 0 0"/>
